File: PCB-dyb.kicad_sch (KiCad schematic)
At the start: 5 parts, among them U1 74AUC2G08, U2 74AUC2G08, U3 74AUC2G04, U4 74AUC2G04, U5 74AUC2G04

Commit message: Somme 2*4bits
Parts:
- removed U1, U2: 74AUC2G08, symbol 74xGxx:74AUC2G08
- removed U3, U4, U5: 74AUC2G04, symbol 74xGxx:74AUC2G04
- added U1: 74AHC1G86, symbol 74xGxx:74AHC1G86
- added U10, U3, U7: (no value), Package_Sorën:SOIC-14_3.9x8.7mm_P1.27mm, symbol CornetPrisme_Library:SN74ALVC08DR
- added U11, U4, U8: 74LVC1G386, symbol 74xGxx:74LVC1G386
- added U2: 74AHC1G08, symbol 74xGxx:74AHC1G08
- added U5, U6, U9: 74LVC1G332, symbol 74xGxx:74LVC1G332
Connections:
- new net: U6.3, U7.3 (4Y)
- new net: U6.6, U7.11 (4Y)
- new net: U10.8 (4Y), U9.1
- new net: U10.3 (4Y), U9.3
- new net: U10.11 (4Y), U9.6
- new net: U6.1, U7.8 (4Y)
- new net: U3.8 (4Y), U5.1
- new net: U3.3 (4Y), U5.3
- new net: U3.11 (4Y), U5.6
- new net C0: U2.4, U3.10 (4B), U3.13 (4B), U4.6
- new net C1: U5.4, U7.10 (4B), U7.13 (4B), U8.6
- new net C2: U10.10 (4B), U10.13 (4B), U11.6, U6.4
- new net S0: U1.4
- new net S1: U4.4
- new net S2: U8.4
- new net S3: U11.4
- new net S4: U9.4
- new net b0: U10.1 (4A), U10.12 (4A), U11.1
- new net b1: U10.2 (4B), U10.9 (4A), U11.3
- new net c0: U7.1 (4A), U7.12 (4A), U8.1
- new net c1: U7.2 (4B), U7.9 (4A), U8.3
- new net d0: U3.1 (4A), U3.12 (4A), U4.1
- new net d1: U3.2 (4B), U3.9 (4A), U4.3
- new net e0: U1.1, U2.1
- new net e1: U1.2, U2.2

Commit message: Add : adder logic
Parts:
- removed U1: 74AHC1G86, symbol 74xGxx:74AHC1G86
- removed U10, U3, U7: (no value), Package_Sorën:SOIC-14_3.9x8.7mm_P1.27mm, symbol CornetPrisme_Library:SN74ALVC08DR
- removed U11, U4, U8: 74LVC1G386, symbol 74xGxx:74LVC1G386
- removed U2: 74AHC1G08, symbol 74xGxx:74AHC1G08
- removed U5, U6, U9: 74LVC1G332, symbol 74xGxx:74LVC1G332
Other:
- added sheet Adder Logic (adder-logic.kicad_sch)
- added sheet Tens Logic (tens-logic.kicad_sch)

Commit message: modify : Units Logic
Other:
- added sheet Units Logic (units-logic.kicad_sch)
Changed lines of the file:
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@@
+	)
+	(sheet
+		(at 317.5 50.8)
+		(size 12.7 12.7)
+		(exclude_from_sim no)
+		(in_bom yes)
+		(on_board yes)
+		(dnp no)
+		(fields_autoplaced yes)
+		(stroke
+			(width 0.1524)
+			(type solid)
+		)
+		(fill
+			(color 0 0 0 0)
+		)
+		(property "Sheetname" "Units Logic"
+			(at 317.5 50.0884 0)
+			(show_name no)
+			(do_not_autoplace no)
+			(effects
+				(font
+					(size 1.27 1.27)
+				)
+				(justify left bottom)
+			)
+		)
+		(property "Sheetfile" "units-logic.kicad_sch"
+			(at 317.5 64.0846 0)
+			(show_name no)
+			(do_not_autoplace no)
+			(effects
+				(font
+					(size 1.27 1.27)
+				)
+				(justify left top)
+			)
+		)
+		(instances
+			(project "PCB-dyb"
+				(path "/14e8619a-6057-40b5-87f2-cdde3077dc07"
+					(page "4")
+				)
+			)
+		)
 	)
 	(sheet

Commit message: add : alimentation
Parts:
- added BT1: Battery_Cell, symbol Device:Battery_Cell
- added C17, C37: 1u, symbol Device:C
- added D1: ESD131-B1-W0201, Diode_SMD:Infineon_SG-WLL-2-3_0.58x0.28_P0.36mm, symbol Diode:ESD131-B1-W0201
- added J1, J2: Conn_01x10, symbol Connector_Generic:Conn_01x10
- added SW1: SW_SPDT, symbol Switch:SW_SPDT
- added TP1, TP2, TP3: TestPoint, symbol Connector:TestPoint
- added U49: TPS7A20xxxDBV, Package_TO_SOT_SMD:SOT-23-5, symbol Regulator_Linear:TPS7A20xxxDBV
Connections:
- new net: BT1.1 (+), D1.2 (A2), SW1.3 (C)
- new net: C17.2, U49.1 (IN), U49.3 (EN)
- new net +1V8: C37.1, TP1.1, U49.5 (OUT)
- new net +BATT: C17.1, SW1.2 (B), TP3.1
- new net GND: BT1.2 (-), C37.2, D1.1 (A1), SW1.1 (A), TP2.1, U49.2 (GND)
Other:
- sheet Adder Logic ports: added a2, b0, b1, b2, c0, c1, c2, d0, d1, d2, e0, e1, e2; removed none
- sheet Tens Logic ports: added D_1, D_2, D_3, a2, b2, c2, d2; removed none
- sheet Units Logic ports: added U_1, U_2, U_3, U_4, a2, b2, c2, d2, e2; removed none
- note added: "CR2032"
- note added: "LDO"

Commit message: add : connection
Connections:
- net GND: now also J1.10 (Pin_10)
- net Tens Logic/D_1: now also J1.3 (Pin_3)
- net Tens Logic/D_2: now also J1.2 (Pin_2)
- net Tens Logic/D_3: now also J1.1 (Pin_1)
- net Units Logic/U_1: now also J1.8 (Pin_8)
- net Units Logic/U_2: now also J1.7 (Pin_7)
- net Units Logic/U_3: now also J1.6 (Pin_6)
- net Units Logic/U_4: now also J1.5 (Pin_5)

Commit message: Branchement des pins
Parts:
- added D10, D11, D12, D13, D14, D2, D3, D4, D5, D6, D7, D8, D9: ESD131-B1-W0201, Diode_SMD:Infineon_SG-WLL-2-3_0.58x0.28_P0.36mm, symbol Diode:ESD131-B1-W0201
Connections:
- net Adder Logic/a2: now also D2.2 (A2)
- net Adder Logic/b0: now also D10.1 (A1)
- net Adder Logic/b1: now also D14.1 (A1)
- net Adder Logic/b2: now also D3.2 (A2)
- net Adder Logic/c0: now also D9.1 (A1)
- net Adder Logic/c1: now also D13.1 (A1)
- net Adder Logic/c2: now also D4.2 (A2)
- net Adder Logic/d0: now also D8.1 (A1)
- net Adder Logic/d1: now also D12.1 (A1)
- net Adder Logic/d2: now also D5.2 (A2)
- net Adder Logic/e0: now also D7.1 (A1)
- net Adder Logic/e1: now also D11.1 (A1)
- net Adder Logic/e2: now also D6.2 (A2)
- net GND: now also J2.10 (Pin_10)
- net Tens Logic/D_1: now also J1.4 (Pin_4); no longer J1.3 (Pin_3)
- net Tens Logic/D_2: now also J1.3 (Pin_3); no longer J1.2 (Pin_2)
- net Tens Logic/D_3: now also J1.2 (Pin_2); no longer J1.1 (Pin_1)
- net at J2.1 (Pin_1): now also D7.2 (A2)
- net at J2.2 (Pin_2): now also D8.2 (A2)
- net at J2.3 (Pin_3): now also D9.2 (A2)
- net at J2.4 (Pin_4): now also D10.2 (A2)
- net at J2.5 (Pin_5): now also D11.2 (A2)
- net at J2.6 (Pin_6): now also D12.2 (A2)
- net at J2.7 (Pin_7): now also D13.2 (A2)
- net at J2.8 (Pin_8): now also D14.2 (A2)
- new net a2: D2.1 (A1)
- new net b2: D3.1 (A1)
- new net c2: D4.1 (A1)
- new net d2: D5.1 (A1)
- new net e2: D6.1 (A1)
- no-connect marks 0 -> 3
Other:
- note added: "System"
- note added: "input"
- note added: "output"
- moved on the sheet: J2

Commit message: ajout composants
Parts:
- removed D10, D11, D12, D13, D14: ESD131-B1-W0201, Diode_SMD:Infineon_SG-WLL-2-3_0.58x0.28_P0.36mm, symbol Diode:ESD131-B1-W0201
- BT1: Basic (none) -> X; JLCPCB Part # (none) -> C964792; Manufacturer (none) -> MYOUNG; Manufacturer Part Number (none) -> BS-08-B2AA016
- C17, C37: Basic (none) -> Y; JLCPCB Part # (none) -> C1592; Manufacturer (none) -> Samsung Electro-Mechanics; Manufacturer Part Number (none) -> CL10A105KO8NNNC
- D1, D2, D3, D4, D5, D6, D7, D8, D9: Basic (none) -> X; JLCPCB Part # (none) -> C20611048; Manufacturer (none) -> TI; Manufacturer Part Number (none) -> TSD05CDYFR
- SW1: Basic (none) -> X; JLCPCB Part # (none) -> C431540; Manufacturer (none) -> SHOU HAN; Manufacturer Part Number (none) -> MSK12C02
- U49: Basic (none) -> X; JLCPCB Part # (none) -> C963430; Manufacturer (none) -> TI; Manufacturer Part Number (none) -> TPS7A2018PDBVR
Connections:
- net Adder Logic/c0 is gone; now on net GND: D9.1 (A1)
- net Adder Logic/d0 is gone; now on net GND: D8.1 (A1)
- net Adder Logic/d2 is gone; now on net b0: D5.2 (A2)
- net Adder Logic/e0 is gone; now on net GND: D7.1 (A1)
- net Adder Logic/e2 is gone; now on net e1: D6.2 (A2)
- net +BATT: now also U49.1 (IN), U49.3 (EN)
- net GND: now also C17.2, D2.1 (A1), D3.1 (A1), D4.1 (A1), D5.1 (A1), D6.1 (A1)
- net a2: no longer D2.1 (A1)
- net b2: no longer D3.1 (A1)
- net c2: no longer D4.1 (A1)
- net d2: no longer D5.1 (A1)
- net e2: no longer D6.1 (A1)
- net c1: now reaches D8.2 (A2)
- net c1: now also J2.7 (Pin_7); no longer J2.2 (Pin_2)
- net e1: now reaches J2.5 (Pin_5)
- net d1: now reaches D7.2 (A2)
- net d1: now also J2.6 (Pin_6); no longer J2.1 (Pin_1)
- net b1: now reaches D9.2 (A2)
- net b1: now also J2.8 (Pin_8); no longer J2.3 (Pin_3)
- net b0: now reaches J2.4 (Pin_4)
- net Adder Logic/a2: no longer names the net of D2.2 (A2)
- net Adder Logic/b2: no longer names the net of D3.2 (A2)
- net Adder Logic/c2: no longer names the net of D4.2 (A2)
- new net c0: J2.3 (Pin_3)
- new net d0: J2.2 (Pin_2)
- new net e0: J2.1 (Pin_1)
Other:
- note added: "protection"
- moved on the sheet: C17

Commit message: elimination of the error in the logic of the tens place
Connections:
- net Tens Logic/D_3: no longer names the net of J1.2 (Pin_2)
- no-connect marks 3 -> 4
Other:
- sheet Tens Logic ports: added none; removed D_3
Changed lines of the file:
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@@
 	)
 	(no_connect
+		(at 177.8 73.66)
+	)
+	(no_connect
 		(at 177.8 91.44)
 	)
@@
 	(wire
 		(pts
-			(xy 158.75 73.66) (xy 177.8 73.66)
-		)
-		(stroke
-			(width 0)
-			(type default)
-		)
-	)
-	(wire
-		(pts
 			(xy 134.62 90.17) (xy 138.43 90.17)
 		)
@@
 			(effects
 				(font
-					(size 1.27 1.27)
-				)
-				(justify right)
-			)
-		)
-		(pin "D_3" output
-			(at 158.75 73.66 0)
-			(effects
-				(font
