File: adder-logic.kicad_sch (KiCad schematic)
At the start: 11 parts, among them U12 74LVC1G332, U16 74LVC1G386, U17 74LVC1G332, U18 74LVC1G386, U19 74LVC1G332, U20 74LVC1G386, U21 74AHC1G08, U22 74AHC1G86

Commit message: add : alimentation
Parts:
- added C1, C10, C11, C12, C2, C3, C4, C6, C7, C8, C9: 0.1u, symbol Device:C
Connections:
- net e0: now also U21.2; no longer U21.1
- net e1: now also U21.1; no longer U21.2
- net +1V8: now reaches U14.14 (VCC)
- net +1V8: now also U12.5 (VCC), U13.14 (VCC), U15.14 (VCC), U16.5 (VCC), U17.5 (VCC), U18.5 (VCC), U19.5 (VCC), U20.5 (VCC), U21.5 (VCC), U22.5 (VCC), C1.1, C10.1, C11.1, C12.1, C2.1, C3.1, C4.2, C6.2, C7.1, C8.2, C9.2
- net GND: now reaches U14.7 (GND)
- net GND: now also U12.2 (GND), U13.7 (GND), U15.7 (GND), U16.2 (GND), U17.2 (GND), U18.2 (GND), U19.2 (GND), U20.2 (GND), U21.3 (GND), U22.3 (GND), C1.2, C10.2, C11.2, C12.2, C2.2, C3.2, C4.1, C6.1, C7.2, C8.1, C9.1
- net at U12.3: now also U13.11 (4Y); no longer U13.3 (1Y)
- net at U12.6: now also U13.3 (1Y); no longer U13.11 (4Y)
- net at U17.3: now also U14.11 (4Y); no longer U14.3 (1Y)
- net at U17.6: now also U14.3 (1Y); no longer U14.11 (4Y)
- net at U15.11 (4Y): now also U19.3; no longer U19.6
- net at U15.3 (1Y): now also U19.6; no longer U19.3
Other:
- moved on the sheet: U12, U17, U19, U21, U22

Commit message: Branchement des pins
Connections:
- no-connect marks 0 -> 9

Commit message: ajout composants
Parts:
- C1, C10, C11, C12, C2, C3, C4, C6, C7, C8, C9: Basic (none) -> Y; JLCPCB Part # (none) -> C1591; Manufacturer (none) -> Samsung Electro-Mechanics; Manufacturer Part Number (none) -> CL10B104KB8NNNC
- U12, U17, U19: Basic (none) -> X; JLCPCB Part # (none) -> C43368; Manufacturer (none) -> TI; Manufacturer Part Number (none) -> SN74LVC1G332DBVR
- U13, U14, U15: Basic (none) -> X; JLCPCB Part # (none) -> C2868761; Manufacturer (none) -> TI; Manufacturer Part Number (none) -> SN74ALVC08DR
- U16, U18, U20: Basic (none) -> X; JLCPCB Part # (none) -> C2867271; Manufacturer (none) -> TI; Manufacturer Part Number (none) -> SN74LVC1G386DCKR
- U21: Basic (none) -> X; JLCPCB Part # (none) -> C2863707; Manufacturer (none) -> TI; Manufacturer Part Number (none) -> SN74AUC1G08DCKR
- U22: Basic (none) -> X; JLCPCB Part # (none) -> C2869047; Manufacturer (none) -> TI; Manufacturer Part Number (none) -> SN74AUC1G86DCKR

Commit message: add footprint
Parts:
- C1, C10, C11, C12, C2, C3, C4, C6, C7, C8, C9: footprint (none) -> Capacitor_SMD:C_0603_1608Metric
- U12, U17, U19: footprint (none) -> Package_TO_SOT_SMD:SOT-23-6
- U16, U18, U20: footprint (none) -> Package_TO_SOT_SMD:Texas_R-PDSO-G6
- U21, U22: footprint (none) -> Package_TO_SOT_SMD:SOT-353_SC-70-5
Changed lines of the file:
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@@
 			)
 		)
-		(property "Footprint" ""
+		(property "Footprint" "Capacitor_SMD:C_0603_1608Metric"
 			(at 41.91 152.7048 0)
 			(hide yes)
@@
 			)
 		)
-		(property "Footprint" ""
+		(property "Footprint" "Capacitor_SMD:C_0603_1608Metric"
 			(at 217.4748 86.36 0)
 			(hide yes)
@@
 			)
 		)
-		(property "Footprint" ""
+		(property "Footprint" "Package_TO_SOT_SMD:Texas_R-PDSO-G6"
 			(at 139.7 86.36 0)
 			(hide yes)
@@
 			)
 		)
-		(property "Footprint" ""
+		(property "Footprint" "Package_TO_SOT_SMD:Texas_R-PDSO-G6"
 			(at 72.39 86.36 0)
 			(hide yes)
@@
 			)
 		)
-		(property "Footprint" ""
+		(property "Footprint" "Package_TO_SOT_SMD:Texas_R-PDSO-G6"
 			(at 208.28 86.36 0)
 			(hide yes)
@@
 			)
 		)
-		(property "Footprint" ""
+		(property "Footprint" "Package_TO_SOT_SMD:SOT-23-6"
 			(at 27.94 50.8 0)
 			(hide yes)
@@
 			)
 		)
-		(property "Footprint" ""
+		(property "Footprint" "Capacitor_SMD:C_0603_1608Metric"
 			(at 156.21 41.6052 0)
 			(hide yes)
@@
 			)
 		)
-		(property "Footprint" ""
+		(property "Footprint" "Package_TO_SOT_SMD:SOT-23-6"
 			(at 95.25 50.8 0)
 			(hide yes)
@@
 			)
 		)
-		(property "Footprint" ""
+		(property "Footprint" "Capacitor_SMD:C_0603_1608Metric"
 			(at 150.8252 93.98 0)
 			(hide yes)
@@
 			)
 		)
-		(property "Footprint" ""
+		(property "Footprint" "Capacitor_SMD:C_0603_1608Metric"
 			(at 20.32 41.6052 0)
 			(hide yes)
@@
 			)
 		)
-		(property "Footprint" ""
+		(property "Footprint" "Package_TO_SOT_SMD:SOT-353_SC-70-5"
 			(at 234.95 62.23 0)
 			(hide yes)
@@
 			)
 		)
-		(property "Footprint" ""
+		(property "Footprint" "Capacitor_SMD:C_0603_1608Metric"
 			(at 242.57 51.1048 0)
 			(hide yes)
@@
 			)
 		)
-		(property "Footprint" ""
+		(property "Footprint" "Capacitor_SMD:C_0603_1608Metric"
 			(at 81.5848 86.36 0)
 			(hide yes)
@@
 			)
 		)
-		(property "Footprint" ""
+		(property "Footprint" "Capacitor_SMD:C_0603_1608Metric"
 			(at 95.25 39.6748 0)
 			(hide yes)
@@
 			)
 		)
-		(property "Footprint" ""
+		(property "Footprint" "Capacitor_SMD:C_0603_1608Metric"
 			(at 87.63 152.7048 0)
 			(hide yes)
@@
 			)
 		)
-		(property "Footprint" ""
+		(property "Footprint" "Capacitor_SMD:C_0603_1608Metric"
 			(at 63.5 152.7048 0)
 			(hide yes)
@@
 			)
 		)
-		(property "Footprint" ""
+		(property "Footprint" "Package_TO_SOT_SMD:SOT-353_SC-70-5"
 			(at 262.89 82.55 0)
 			(hide yes)
@@
 			)
 		)
-		(property "Footprint" ""
+		(property "Footprint" "Package_TO_SOT_SMD:SOT-23-6"
 			(at 163.83 50.8 0)
 			(hide yes)
@@
 			)
 		)
-		(property "Footprint" ""
+		(property "Footprint" "Capacitor_SMD:C_0603_1608Metric"
 			(at 272.0848 82.55 0)
 			(hide yes)
