File: PCB-dyb.kicad_pcb (KiCad board)
At the start: 2 copper layers, 93 parts, among them J1 Conn_01x10, J2 Conn_01x10, SW1 SW_SPDT, U12 74LVC1G332, U16 74LVC1G386, U17 74LVC1G332, U18 74LVC1G386, U19 74LVC1G332, U20 74LVC1G386, U21 74AHC1G08, U22 74AHC1G86, U23 74AUC2G04, U24 ², U26 ², U27 ², U30 ², U31 ², U34 ², U35 ², U37 74AUC2G08, U38 ², U49 TPS7A20xxxDBV, U5 74AUC2G04, U6 74AUC2G04, U7 74AUC2G04

Commit message: dbt disposition
Parts:
- moved J2 98.2 mm to (20.2, 84.4)
- moved C11 95.0 mm to (21.0, 122.3)
- moved C4 95.0 mm to (17.0, 122.3)
- moved C7 95.0 mm to (17.0, 127.3)
- moved C8 95.0 mm to (21.0, 114.7)
- moved C12 95.0 mm to (21.0, 124.8)
- moved C6 95.0 mm to (17.0, 124.8)
- moved C1 94.6 mm to (17.0, 114.2)
- moved C2 94.4 mm to (17.0, 116.5)
- moved C3 94.4 mm to (17.0, 119.0)
- moved U22 84.9 mm to (31.7, 105.7)
- moved U21 83.4 mm to (31.5, 100.2)
- moved U15 80.2 mm to (35.5, 91.0)
- moved U12 78.0 mm to (104.6, 99.5)
- moved U14 77.5 mm to (72.8, 100.8)
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
Commit message: dbt layout
Parts:
- moved J1 185.0 mm to (271.5, 116.0)
- moved C17 125.7 mm to (30.4, 185.2)
- moved C37 125.7 mm to (30.4, 187.7)
- moved D1 125.7 mm to (16.5, 196.7)
- moved SW1 125.7 mm to (23.4, 187.4)
- moved U49 125.7 mm to (27.6, 193.4)
- moved C38 120.8 mm to (170.1, 107.6)
- moved C40 120.8 mm to (170.1, 110.1)
- moved C41 120.8 mm to (170.1, 112.6)
- moved C42 120.8 mm to (170.1, 115.1)
- moved C43 120.8 mm to (170.1, 117.6)
- moved C44 120.8 mm to (170.1, 120.2)
- moved C45 120.8 mm to (174.2, 107.6)
- moved C46 120.8 mm to (174.2, 110.1)
- moved C47 120.8 mm to (174.2, 112.6)
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Routing:
- net /e0: track 0.00 -> 8.64 mm
- net /d0: track 0.00 -> 8.29 mm
- net /e1: track 0.00 -> 7.95 mm
- net /c0: track 0.00 -> 7.95 mm
- net /d1: track 0.00 -> 7.77 mm
- net /b0: track 0.00 -> 7.74 mm
- net /c1: track 0.00 -> 7.69 mm
- net /b1: track 0.00 -> 7.46 mm

Commit message: dbt positionnement
Parts:
- removed C31: 0.1u, Capacitor_SMD:C_0603_1608Metric
- removed U28: ~, Package_TO_SOT_SMD:SOT-23-6
- moved D1 118.8 mm to (26.4, 78.3)
- moved C17 115.8 mm to (34.6, 69.5)
- moved C37 115.8 mm to (34.6, 72.0)
- moved U49 115.8 mm to (31.8, 77.7)
- moved SW1 115.8 mm to (27.6, 71.7)
- moved U38 84.6 mm to (148.1, 126.5)
- moved U37 72.0 mm to (132.7, 117.3)
- moved C27 71.1 mm to (148.0, 122.8)
- moved C28 71.0 mm to (104.5, 75.3)
- moved U31 70.0 mm to (129.4, 101.3)
- moved J1 67.4 mm to (206.0, 131.7)
- moved C12 65.5 mm to (80.2, 29.5), turned to 180 degrees
- moved U30 65.4 mm to (117.9, 88.0)
- moved C3 65.0 mm to (74.5, 21.5), turned to 180 degrees
- moved U11 64.6 mm to (109.4, 80.6)
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Routing:
- net /e0: track 8.64 -> 0.00 mm
- net /d0: track 8.29 -> 0.00 mm
- net /e1: track 7.95 -> 0.00 mm
- net /c0: track 7.95 -> 0.00 mm
- net /d1: track 7.77 -> 0.00 mm
- net /b0: track 7.74 -> 0.00 mm
- net /c1: track 7.69 -> 0.00 mm
- net /b1: track 7.46 -> 0.00 mm
